File: alt-Lab2/ArduinoClock/ArduinoClock.sch (EAGLE design)
At the start: 36 parts, among them IC1 DS3231/SO, U1 MIC5225-5.0, U2 ATMEGA328P, U3 CP2104, U4 MIC5225-3.3, X1 20329, Y2 CSTCE16M0V53-R0 16MHZ

Commit message: fixed some ground planes and airwired
Parts:
- removed FD1, FD2: FIDUCIAL"", microbuilder:FIDUCIAL""
Changed lines of the file:
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@@
 <part name="GND14" library="supply1" deviceset="GND" device=""/>
 <part name="P+5" library="supply1" deviceset="+5V" device=""/>
-<part name="FD1" library="microbuilder" deviceset="FIDUCIAL" device="&quot;&quot;"/>
-<part name="FD2" library="microbuilder" deviceset="FIDUCIAL" device="&quot;&quot;"/>
 <part name="GND11" library="supply1" deviceset="GND" device=""/>
 <part name="C4" library="microbuilder" deviceset="CAP_CERAMIC" device="0805-NOOUTLINE" value="0.1uF"/>
@@
 <attribute name="VALUE" x="375.285" y="231.14" size="1.778" layer="96" rot="R180"/>
 </instance>
-<instance part="FD1" gate="G$1" x="375.92" y="27.94" smashed="yes"/>
-<instance part="FD2" gate="G$1" x="381" y="27.94" smashed="yes"/>
 <instance part="GND11" gate="1" x="231.14" y="208.28" smashed="yes">
 <attribute name="VALUE" x="228.6" y="205.74" size="1.778" layer="96"/>
